File: naive_business_card.kicad_sch (KiCad schematic)
At the start: 14 parts, among them Q1 2N3904, SW1 DS01-254-S-01BE, U1 TLC555IP

Commit message: Rename repo
Parts:
- BT1: footprint business_card:BAT-HLD-001-THM -> naive_business_card:BAT-HLD-001-THM; symbol business_card:BAT-HLD-001-THM -> naive_business_card:BAT-HLD-001-THM
- Q1: footprint business_card:2N3904 -> naive_business_card:2N3904
- RV1: footprint business_card:3306P-1-504 -> naive_business_card:3306P-1-504
- SW1: footprint business_card:DS01-254-S-01BE -> naive_business_card:DS01-254-S-01BE; symbol business_card:DS01-254-S-01BE -> naive_business_card:DS01-254-S-01BE
- U1: footprint business_card:TLC555IP -> naive_business_card:TLC555IP; symbol business_card:TLC555IP -> naive_business_card:TLC555IP
Changed lines of the file:
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@@
 		)
 		(instances
-			(project "business_card"
+			(project "naive_business_card"
 				(path "/b84feb65-b9c7-4def-9ca7-9e4ec7b305d8"
 					(reference "#PWR01")
@@
 		)
 		(instances
-			(project "business_card"
+			(project "naive_business_card"
 				(path "/b84feb65-b9c7-4def-9ca7-9e4ec7b305d8"
 					(reference "#PWR06")
@@
 	)
 	(symbol
-		(lib_id "business_card:BAT-HLD-001-THM")
+		(lib_id "naive_business_card:BAT-HLD-001-THM")
 		(at 82.55 121.92 0)
 		(unit 1)
@@
 			)
 		)
-		(property "Footprint" "business_card:BAT-HLD-001-THM"
+		(property "Footprint" "naive_business_card:BAT-HLD-001-THM"
 			(at 82.55 121.92 0)
 			(effects
@@
 		)
 		(instances
-			(project "business_card"
+			(project "naive_business_card"
 				(path "/b84feb65-b9c7-4def-9ca7-9e4ec7b305d8"
 					(reference "#FLG01")
@@
 		)
 		(instances
-			(project "business_card"
+			(project "naive_business_card"
 				(path "/b84feb65-b9c7-4def-9ca7-9e4ec7b305d8"
 					(reference "#PWR08")
@@
 		)
 		(instances
-			(project "business_card"
+			(project "naive_business_card"
 				(path "/b84feb65-b9c7-4def-9ca7-9e4ec7b305d8"
 					(reference "#PWR09")
@@
 		)
 		(instances
-			(project "business_card"
+			(project "naive_business_card"
 				(path "/b84feb65-b9c7-4def-9ca7-9e4ec7b305d8"
 					(reference "R4")
@@
 			)
 		)
-		(property "Footprint" "business_card:2N3904"
+		(property "Footprint" "naive_business_card:2N3904"
 			(at 119.38 123.825 0)
 			(effects
@@
 		)
 		(instances
-			(project "business_card"
+			(project "naive_business_card"
 				(path "/b84feb65-b9c7-4def-9ca7-9e4ec7b305d8"
 					(reference "Q1")
@@
 		)
 		(instances
-			(project "business_card"
+			(project "naive_business_card"
 				(path "/b84feb65-b9c7-4def-9ca7-9e4ec7b305d8"
 					(reference "C2")
@@
 	)
 	(symbol
-		(lib_id "business_card:TLC555IP")
+		(lib_id "naive_business_card:TLC555IP")
 		(at 146.05 101.6 0)
 		(unit 1)
@@
 			)
 		)
-		(property "Footprint" "business_card:TLC555IP"
+		(property "Footprint" "naive_business_card:TLC555IP"
 			(at 146.05 101.6 0)
 			(effects
@@
 		)
 		(instances
-			(project "business_card"
+			(project "naive_business_card"
 				(path "/b84feb65-b9c7-4def-9ca7-9e4ec7b305d8"
 					(reference "U1")
@@
 		)
 		(instances
-			(project "business_card"
+			(project "naive_business_card"
 				(path "/b84feb65-b9c7-4def-9ca7-9e4ec7b305d8"
 					(reference "R5")
@@
 		)
 		(instances
-			(project "business_card"
+			(project "naive_business_card"
 				(path "/b84feb65-b9c7-4def-9ca7-9e4ec7b305d8"
 					(reference "R2")
@@
 		)
 		(instances
-			(project "business_card"
+			(project "naive_business_card"
 				(path "/b84feb65-b9c7-4def-9ca7-9e4ec7b305d8"
 					(reference "#PWR04")
@@
 		)
 		(instances
-			(project "business_card"
+			(project "naive_business_card"
 				(path "/b84feb65-b9c7-4def-9ca7-9e4ec7b305d8"
 					(reference "R1")
@@
 		)
 		(instances
-			(project "business_card"
+			(project "naive_business_card"
 				(path "/b84feb65-b9c7-4def-9ca7-9e4ec7b305d8"
 					(reference "#PWR07")
@@
 		)
 		(instances
-			(project "business_card"
+			(project "naive_business_card"
 				(path "/b84feb65-b9c7-4def-9ca7-9e4ec7b305d8"
 					(reference "C1")
@@
 		)
 		(instances
-			(project "business_card"
+			(project "naive_business_card"
 				(path "/b84feb65-b9c7-4def-9ca7-9e4ec7b305d8"
 					(reference "R3")
@@
 		)
 		(instances
-			(project "business_card"
+			(project "naive_business_card"
 				(path "/b84feb65-b9c7-4def-9ca7-9e4ec7b305d8"
 					(reference "#PWR02")
@@
 		)
 		(instances
-			(project "business_card"
+			(project "naive_business_card"
 				(path "/b84feb65-b9c7-4def-9ca7-9e4ec7b305d8"
 					(reference "#PWR05")
@@
 		)
 		(instances
-			(project "business_card"
+			(project "naive_business_card"
 				(path "/b84feb65-b9c7-4def-9ca7-9e4ec7b305d8"
 					(reference "D1")
@@
 			)
 		)
-		(property "Footprint" "business_card:3306P-1-504"
+		(property "Footprint" "naive_business_card:3306P-1-504"
 			(at 171.45 116.84 0)
 			(effects
@@
 		)
 		(instances
-			(project "business_card"
+			(project "naive_business_card"
 				(path "/b84feb65-b9c7-4def-9ca7-9e4ec7b305d8"
 					(reference "RV1")
@@
 		)
 		(instances
-			(project "business_card"
+			(project "naive_business_card"
 				(path "/b84feb65-b9c7-4def-9ca7-9e4ec7b305d8"
 					(reference "D2")
@@
 	)
 	(symbol
-		(lib_id "business_card:DS01-254-S-01BE")
+		(lib_id "naive_business_card:DS01-254-S-01BE")
 		(at 96.52 105.41 90)
 		(unit 1)
@@
 			)
 		)
-		(property "Footprint" "business_card:DS01-254-S-01BE"
+		(property "Footprint" "naive_business_card:DS01-254-S-01BE"
 			(at 96.52 105.41 0)
 			(effects
@@
 		)
 		(instances
-			(project "business_card"
+			(project "naive_business_card"
 				(path "/b84feb65-b9c7-4def-9ca7-9e4ec7b305d8"
 					(reference "SW1")
@@
 		)
 		(instances
-			(project "business_card"
+			(project "naive_business_card"
 				(path "/b84feb65-b9c7-4def-9ca7-9e4ec7b305d8"
 					(reference "#PWR03")
