File: naive-business-card.kicad_pcb (KiCad board)
At the start: 2 copper layers, 88.9 x 50.8 mm, 14 parts, among them Q1 2N3904, SW1 DS01-254-S-01BE, U1 TLC555IP

Commit message: Rename the repo
Parts:
- BT1: footprint naive_business_card:BAT-HLD-001-THM -> naive-business-card:BAT-HLD-001-THM
- Q1: footprint naive_business_card:2N3904 -> naive-business-card:2N3904
- RV1: footprint naive_business_card:3306P-1-504 -> naive-business-card:3306P-1-504
- SW1: footprint naive_business_card:DS01-254-S-01BE -> naive-business-card:DS01-254-S-01BE
- U1: footprint naive_business_card:TLC555IP -> naive-business-card:TLC555IP
Changed lines of the file:
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@@
 		(property ki_fp_filters "LED* LED_SMD:* LED_THT:*")
 		(sheetname "Root")
-		(sheetfile "naive_business_card.kicad_sch")
+		(sheetfile "naive-business-card.kicad_sch")
 		(attr through_hole)
 		(fp_line
@@
 		(property ki_fp_filters "CP_*")
 		(sheetname "Root")
-		(sheetfile "naive_business_card.kicad_sch")
+		(sheetfile "naive-business-card.kicad_sch")
 		(attr through_hole)
 		(fp_line
@@
 		(property ki_fp_filters "CP_*")
 		(sheetname "Root")
-		(sheetfile "naive_business_card.kicad_sch")
+		(sheetfile "naive-business-card.kicad_sch")
 		(attr through_hole)
 		(fp_line
@@
 		(property ki_fp_filters "R_*")
 		(sheetname "Root")
-		(sheetfile "naive_business_card.kicad_sch")
+		(sheetfile "naive-business-card.kicad_sch")
 		(attr through_hole)
 		(fp_line
@@
 		)
 	)
-	(footprint "naive_business_card:BAT-HLD-001-THM"
+	(footprint "naive-business-card:BAT-HLD-001-THM"
 		(layer "F.Cu")
 		(at 118.85 116.05 -90)
@@
 			)
 		)
-		(property "Footprint" "naive_business_card:BAT-HLD-001-THM"
+		(property "Footprint" "naive-business-card:BAT-HLD-001-THM"
 			(at 0 0 -90)
 			(unlocked yes)
@@
 		)
 		(sheetname "Root")
-		(sheetfile "naive_business_card.kicad_sch")
+		(sheetfile "naive-business-card.kicad_sch")
 		(attr through_hole)
 		(fp_line
@@
 		(property ki_fp_filters "R_*")
 		(sheetname "Root")
-		(sheetfile "naive_business_card.kicad_sch")
+		(sheetfile "naive-business-card.kicad_sch")
 		(attr through_hole)
 		(fp_line
@@
 		(property ki_fp_filters "LED* LED_SMD:* LED_THT:*")
 		(sheetname "Root")
-		(sheetfile "naive_business_card.kicad_sch")
+		(sheetfile "naive-business-card.kicad_sch")
 		(attr through_hole)
 		(fp_line
@@
 		)
 	)
-	(footprint "naive_business_card:2N3904"
+	(footprint "naive-business-card:2N3904"
 		(layer "F.Cu")
 		(at 131 111.96 -90)
@@
 			)
 		)
-		(property "Footprint" "naive_business_card:2N3904"
+		(property "Footprint" "naive-business-card:2N3904"
 			(at 0 0 90)
 			(layer "F.Fab")
@@
 		(property ki_fp_filters "TO?92*")
 		(sheetname "Root")
-		(sheetfile "naive_business_card.kicad_sch")
+		(sheetfile "naive-business-card.kicad_sch")
 		(attr through_hole)
 		(fp_line
@@
 		)
 	)
-	(footprint "naive_business_card:DS01-254-S-01BE"
+	(footprint "naive-business-card:DS01-254-S-01BE"
 		(layer "F.Cu")
 		(at 133.61 124.4 -90)
@@
 			)
 		)
-		(property "Footprint" "naive_business_card:DS01-254-S-01BE"
+		(property "Footprint" "naive-business-card:DS01-254-S-01BE"
 			(at 0 3.62 -90)
 			(unlocked yes)
@@
 		)
 		(sheetname "Root")
-		(sheetfile "naive_business_card.kicad_sch")
+		(sheetfile "naive-business-card.kicad_sch")
 		(attr through_hole)
 		(fp_rect
@@
 		)
 	)
-	(footprint "naive_business_card:TLC555IP"
+	(footprint "naive-business-card:TLC555IP"
 		(layer "F.Cu")
 		(at 162.6375 118.25 -90)
@@
 			)
 		)
-		(property "Footprint" "naive_business_card:TLC555IP"
+		(property "Footprint" "naive-business-card:TLC555IP"
 			(at 0 0 -90)
 			(unlocked yes)
@@
 		)
 		(sheetname "Root")
-		(sheetfile "naive_business_card.kicad_sch")
+		(sheetfile "naive-business-card.kicad_sch")
 		(attr through_hole)
 		(fp_rect
@@
 		(property ki_fp_filters "R_*")
 		(sheetname "Root")
-		(sheetfile "naive_business_card.kicad_sch")
+		(sheetfile "naive-business-card.kicad_sch")
 		(attr through_hole)
 		(fp_line
@@
 		(property ki_fp_filters "R_*")
 		(sheetname "Root")
-		(sheetfile "naive_business_card.kicad_sch")
+		(sheetfile "naive-business-card.kicad_sch")
 		(attr through_hole)
 		(fp_line
@@
 		)
 	)
-	(footprint "naive_business_card:3306P-1-504"
+	(footprint "naive-business-card:3306P-1-504"
 		(layer "F.Cu")
 		(at 178.5 97 -90)
@@
 			)
 		)
-		(property "Footprint" "naive_business_card:3306P-1-504"
+		(property "Footprint" "naive-business-card:3306P-1-504"
 			(at 0 0 -90)
 			(unlocked yes)
@@
 		(property ki_fp_filters "Potentiometer*")
 		(sheetname "Root")
-		(sheetfile "naive_business_card.kicad_sch")
+		(sheetfile "naive-business-card.kicad_sch")
 		(attr through_hole)
 		(fp_line
@@
 		(property ki_fp_filters "R_*")
 		(sheetname "Root")
-		(sheetfile "naive_business_card.kicad_sch")
+		(sheetfile "naive-business-card.kicad_sch")
 		(attr through_hole)
 		(fp_line
