File: naive-business-card.kicad_sch (KiCad schematic)
At the start: 14 parts, among them Q1 2N3904, SW1 DS01-254-S-01BE, U1 TLC555IP

Commit message: Rename the repo
Parts:
- BT1: footprint naive_business_card:BAT-HLD-001-THM -> naive-business-card:BAT-HLD-001-THM; symbol naive_business_card:BAT-HLD-001-THM -> naive-business-card:BAT-HLD-001-THM
- Q1: footprint naive_business_card:2N3904 -> naive-business-card:2N3904
- RV1: footprint naive_business_card:3306P-1-504 -> naive-business-card:3306P-1-504
- SW1: footprint naive_business_card:DS01-254-S-01BE -> naive-business-card:DS01-254-S-01BE; symbol naive_business_card:DS01-254-S-01BE -> naive-business-card:DS01-254-S-01BE
- U1: footprint naive_business_card:TLC555IP -> naive-business-card:TLC555IP; symbol naive_business_card:TLC555IP -> naive-business-card:TLC555IP
Changed lines of the file:
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@@
 		)
 		(instances
-			(project "naive_business_card"
+			(project "naive-business-card"
 				(path "/b84feb65-b9c7-4def-9ca7-9e4ec7b305d8"
 					(reference "#PWR01")
@@
 		)
 		(instances
-			(project "naive_business_card"
+			(project "naive-business-card"
 				(path "/b84feb65-b9c7-4def-9ca7-9e4ec7b305d8"
 					(reference "#PWR06")
@@
 	)
 	(symbol
-		(lib_id "naive_business_card:BAT-HLD-001-THM")
+		(lib_id "naive-business-card:BAT-HLD-001-THM")
 		(at 82.55 121.92 0)
 		(unit 1)
@@
 			)
 		)
-		(property "Footprint" "naive_business_card:BAT-HLD-001-THM"
+		(property "Footprint" "naive-business-card:BAT-HLD-001-THM"
 			(at 82.55 121.92 0)
 			(effects
@@
 		)
 		(instances
-			(project "naive_business_card"
+			(project "naive-business-card"
 				(path "/b84feb65-b9c7-4def-9ca7-9e4ec7b305d8"
 					(reference "#FLG01")
@@
 		)
 		(instances
-			(project "naive_business_card"
+			(project "naive-business-card"
 				(path "/b84feb65-b9c7-4def-9ca7-9e4ec7b305d8"
 					(reference "#PWR08")
@@
 		)
 		(instances
-			(project "naive_business_card"
+			(project "naive-business-card"
 				(path "/b84feb65-b9c7-4def-9ca7-9e4ec7b305d8"
 					(reference "#PWR09")
@@
 		)
 		(instances
-			(project "naive_business_card"
+			(project "naive-business-card"
 				(path "/b84feb65-b9c7-4def-9ca7-9e4ec7b305d8"
 					(reference "R4")
@@
 			)
 		)
-		(property "Footprint" "naive_business_card:2N3904"
+		(property "Footprint" "naive-business-card:2N3904"
 			(at 119.38 123.825 0)
 			(effects
@@
 		)
 		(instances
-			(project "naive_business_card"
+			(project "naive-business-card"
 				(path "/b84feb65-b9c7-4def-9ca7-9e4ec7b305d8"
 					(reference "Q1")
@@
 		)
 		(instances
-			(project "naive_business_card"
+			(project "naive-business-card"
 				(path "/b84feb65-b9c7-4def-9ca7-9e4ec7b305d8"
 					(reference "C2")
@@
 	)
 	(symbol
-		(lib_id "naive_business_card:TLC555IP")
+		(lib_id "naive-business-card:TLC555IP")
 		(at 146.05 101.6 0)
 		(unit 1)
@@
 			)
 		)
-		(property "Footprint" "naive_business_card:TLC555IP"
+		(property "Footprint" "naive-business-card:TLC555IP"
 			(at 146.05 101.6 0)
 			(effects
@@
 		)
 		(instances
-			(project "naive_business_card"
+			(project "naive-business-card"
 				(path "/b84feb65-b9c7-4def-9ca7-9e4ec7b305d8"
 					(reference "U1")
@@
 		)
 		(instances
-			(project "naive_business_card"
+			(project "naive-business-card"
 				(path "/b84feb65-b9c7-4def-9ca7-9e4ec7b305d8"
 					(reference "R5")
@@
 		)
 		(instances
-			(project "naive_business_card"
+			(project "naive-business-card"
 				(path "/b84feb65-b9c7-4def-9ca7-9e4ec7b305d8"
 					(reference "R2")
@@
 		)
 		(instances
-			(project "naive_business_card"
+			(project "naive-business-card"
 				(path "/b84feb65-b9c7-4def-9ca7-9e4ec7b305d8"
 					(reference "#PWR04")
@@
 		)
 		(instances
-			(project "naive_business_card"
+			(project "naive-business-card"
 				(path "/b84feb65-b9c7-4def-9ca7-9e4ec7b305d8"
 					(reference "R1")
@@
 		)
 		(instances
-			(project "naive_business_card"
+			(project "naive-business-card"
 				(path "/b84feb65-b9c7-4def-9ca7-9e4ec7b305d8"
 					(reference "#PWR07")
@@
 		)
 		(instances
-			(project "naive_business_card"
+			(project "naive-business-card"
 				(path "/b84feb65-b9c7-4def-9ca7-9e4ec7b305d8"
 					(reference "C1")
@@
 		)
 		(instances
-			(project "naive_business_card"
+			(project "naive-business-card"
 				(path "/b84feb65-b9c7-4def-9ca7-9e4ec7b305d8"
 					(reference "R3")
@@
 		)
 		(instances
-			(project "naive_business_card"
+			(project "naive-business-card"
 				(path "/b84feb65-b9c7-4def-9ca7-9e4ec7b305d8"
 					(reference "#PWR02")
@@
 		)
 		(instances
-			(project "naive_business_card"
+			(project "naive-business-card"
 				(path "/b84feb65-b9c7-4def-9ca7-9e4ec7b305d8"
 					(reference "#PWR05")
@@
 		)
 		(instances
-			(project "naive_business_card"
+			(project "naive-business-card"
 				(path "/b84feb65-b9c7-4def-9ca7-9e4ec7b305d8"
 					(reference "D1")
@@
 			)
 		)
-		(property "Footprint" "naive_business_card:3306P-1-504"
+		(property "Footprint" "naive-business-card:3306P-1-504"
 			(at 171.45 116.84 0)
 			(effects
@@
 		)
 		(instances
-			(project "naive_business_card"
+			(project "naive-business-card"
 				(path "/b84feb65-b9c7-4def-9ca7-9e4ec7b305d8"
 					(reference "RV1")
@@
 		)
 		(instances
-			(project "naive_business_card"
+			(project "naive-business-card"
 				(path "/b84feb65-b9c7-4def-9ca7-9e4ec7b305d8"
 					(reference "D2")
@@
 	)
 	(symbol
-		(lib_id "naive_business_card:DS01-254-S-01BE")
+		(lib_id "naive-business-card:DS01-254-S-01BE")
 		(at 96.52 105.41 90)
 		(unit 1)
@@
 			)
 		)
-		(property "Footprint" "naive_business_card:DS01-254-S-01BE"
+		(property "Footprint" "naive-business-card:DS01-254-S-01BE"
 			(at 96.52 105.41 0)
 			(effects
@@
 		)
 		(instances
-			(project "naive_business_card"
+			(project "naive-business-card"
 				(path "/b84feb65-b9c7-4def-9ca7-9e4ec7b305d8"
 					(reference "SW1")
@@
 		)
 		(instances
-			(project "naive_business_card"
+			(project "naive-business-card"
 				(path "/b84feb65-b9c7-4def-9ca7-9e4ec7b305d8"
 					(reference "#PWR03")
